File: Pcb/Pcb.sch (KiCad schematic (older format))
At the start: 132 parts, among them J1 TRRS, Q1 2N7002, SW1 SW_Push, SW10 SW_Push, SW11 SW_Push, SW12 SW_Push, SW13 SW_Push, SW14 SW_Push, SW15 SW_Push, SW16 SW_Push, SW17 SW_Push, SW18 SW_Push, SW19 SW_Push, SW2 SW2, SW20 SW_Push, SW21 SW_Push, SW22 SW_Push, SW23 SW_Push, SW24 SW_Push, SW25 SW_Push, SW26 SW_Push, SW27 SW_Push, SW28 SW_Push, SW29 SW_Push, SW3 SW_Push, SW4 SW_Push, SW5 SW_Push, SW6 SW_Push, SW7 SW_Push, SW8 SW_Push, SW9 SW_Push, U1 ProMicro

Commit message: Add support millmax socket for swithes
Parts:
- D1, D10, D11, D12, D13, D14, D15, D16, D17, D18, D19, D2, D20, D21, D22, D23, D24, D25, D26, D27, D28, D3, D4, D5, D6, D7, D8, D9: footprint Used_Footprints:Diode_SMD_TH -> Used_Footprints:Diode_Hybrid_SOD-123
- R1, R10, R11, R12, R13, R14, R15, R16, R17, R18, R19, R2, R20, R21, R22, R23, R24, R25, R26, R27, R28, R29, R3, R30, R31, R4, R5, R6, R7, R8, R9: footprint Used_Footprints:Resistor_SMD_TH -> Used_Footprints:Resistor_Hybrid_0805

Commit message: Replace footprints
Parts:
- R31: value 100k -> 10k
Changed lines of the file:
@@
 P 10200 3025
 F 0 "R31" H 10240 3065 50  0000 L CNN
-F 1 "100k" H 10240 2985 50  0000 L CNN
+F 1 "10k" H 10240 2985 50  0000 L CNN
 F 2 "Used_Footprints:Resistor_Hybrid_0805" H 10200 3025 50  0001 C CNN
 F 3 "~" H 10200 3025 50  0001 C CNN
